Commit message: Update : base_footprint added

File: fusionbot_description/urdf/fusionbot_description.urdf (robot description, URDF)
Before this commit: robot fusionbot, 4 links, 3 joints
Links:
- added link base_footprint
Joints:
- added joint base_link_joint: type fixed, parent base_footprint, child base_link, origin xyz=0 0 0 rpy=0 0 0
